File: hardware/programmer.kicad_pcb (KiCad board)
At the start: 2 copper layers, 11 parts, among them J1 Conn_01x02_Pin, J2 Conn_01x08_Pin, J3 Conn_01x06_Pin, J4 Conn_01x02_Pin, SW1 SW_Push_Dual, SW2 SW_Push_Dual, U2 74HC595, U3 74HC595

Commit message: intial firmware
Parts:
- removed J1, J4: Conn_01x02_Pin, Connector_PinHeader_1.27mm:PinHeader_1x02_P1.27mm_Vertical
- removed J2: Conn_01x08_Pin, Connector_PinHeader_2.54mm:PinHeader_1x08_P2.54mm_Vertical
- removed J3: Conn_01x06_Pin, Connector_PinHeader_2.54mm:PinHeader_1x06_P2.54mm_Vertical
- removed SW1, SW2: SW_Push_Dual, Button_Switch_THT:SW_PUSH_6mm
- added A1: Arduino_UNO_R3, shield-headers:eeprom_programmer, F.Cu at (140.4, 163.1)
- added CLEAR: SW_Push_Dual, Button_Switch_THT:SW_PUSH_6mm, F.Cu at (127.5, 166.6)
- added READ: SW_Push_Dual, Button_Switch_THT:SW_PUSH_6mm, F.Cu at (141.0, 166.8)
- U1: footprint Package_DIP:DIP-28_W15.24mm -> DIP28 _Socket:CONN_110-99-328-41-001000_MIM
- moved U1 121.6 mm to (137.0, 154.1), turned to 180 degrees
- moved C2 65.1 mm to (149.6, 139.1), turned to 180 degrees
- moved U3 50.1 mm to (145.6, 143.6)
- moved U2 48.0 mm to (145.6, 116.5)
- moved C1 22.3 mm to (150.1, 111.7), turned to 180 degrees
Connections:
- net V_{CC} renamed +5V
- U1 pad 1: unconnected-(U1-NC-Pad1) -> RDY/~{BUSY}
- U1 pad 2: A_{12} -> unconnected-(U1-NC-Pad2)
- U1 pad 23: A_{11} -> unconnected-(U1-NC-Pad23)
- U3 pad 3: A_{11} -> unconnected-(U3-QD-Pad3)
- U3 pad 4: A_{12} -> unconnected-(U3-QE-Pad4)
Routing:
- net +5V: track 54.0 -> 110.7 mm
- net CLK: track 49.5 -> 0.00 mm
- net GND: track 122.8 -> 78.5 mm
- net A_{0}: track 0.00 -> 29.0 mm
- net A_{8}: track 0.00 -> 24.8 mm
- net A_{4}: track 0.00 -> 23.2 mm
- net A_{5}: track 0.00 -> 23.0 mm
- net A_{3}: track 0.00 -> 22.7 mm
- net A_{6}: track 0.00 -> 22.7 mm
- net A_{7}: track 0.00 -> 22.4 mm
- net A_{2}: track 0.00 -> 21.9 mm
- net A_{1}: track 0.00 -> 21.6 mm
- net A_{9}: track 0.00 -> 21.3 mm
- net A_{10}: track 0.00 -> 20.3 mm
- net ~{RESET}: track 50.1 -> 42.5 mm
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Other:
- board outline added: 57 x 68.6 mm
- board text removed: "Clear"
- board text removed: "Read"
